File: GAL_8bit_RAM/GAL_8bit_RAM.sch (KiCad schematic (older format))
At the start: 9 parts, among them CN4 HDR-1X12-SIP-100, CN5 HDR-1X12-SIP-100, CN6 HDR-1X12-SIP-100, IC1 74574N, U1 GAL16V8, U2 AS6C4008-55PCN, U3 AS6C4008-55PCN

Commit message: Trying different control line schema
Connections:
- net D10: now also U3.29 (WE#)
- net WE0*: now also U2.29 (WE#)
- net CE* renamed LCE*
- net LCE*: now also U2.22 (CE#)
- net LB* renamed UCE*
- removed net OE*: U1.13 (IO7), U2.24 (OE#), U3.24 (OE#)
- net UB* renamed LOE*
- net LOE*: now also U2.24 (OE#); no longer U2.22 (CE#)
- removed net WE*: U1.14 (IO6), U2.29 (WE#), U3.29 (WE#)
- new net UOE*: U1.14 (IO6), U3.24 (OE#)
Changed lines of the file:
@@
 Text GLabel 4650 5650 0    70   BiDi ~ 0
 WE0*
-Text Label 6250 5400 0    47   ~ 0
-UB*
-Text Label 6250 5500 0    47   ~ 0
-LB*
 Entry Wire Line
 	4700 2350 4800 2450
@@
 Wire Wire Line
 	6850 5200 6850 1800
-Text Label 6250 5300 0    50   ~ 0
-CE*
 Wire Wire Line
 	6600 2450 6900 2450
@@
 Wire Wire Line
 	5600 3750 5600 4400
-Text Label 6250 5600 0    50   ~ 0
-WE*
 Wire Wire Line
 	5250 5700 5100 5700
@@
 	1    0    0    -1
 $EndComp
-Text Label 6250 5700 0    50   ~ 0
-OE*
 Wire Wire Line
 	5250 6000 5250 6350
@@
 RAM_PULL
 Wire Wire Line
-	6250 5400 7250 5400
-Wire Wire Line
-	7250 5400 7250 4300
-Wire Wire Line
-	7250 4300 9550 4300
-Wire Wire Line
-	9550 4300 9550 2600
-Wire Wire Line
-	9550 2600 9300 2600
-Wire Wire Line
-	9350 5850 9750 5850
-Wire Wire Line
-	9750 5850 9750 7350
-Wire Wire Line
-	9750 7350 7050 7350
-Wire Wire Line
-	7050 7350 7050 5500
-Wire Wire Line
-	7050 5500 6250 5500
-Wire Wire Line
-	6250 5600 7350 5600
-Wire Wire Line
-	7350 5600 7350 3900
-Wire Wire Line
-	7350 3900 9300 3900
-Wire Wire Line
-	9300 3900 9300 2800
-Wire Wire Line
-	9300 3900 10200 3900
-Wire Wire Line
-	10200 3900 10200 6050
-Wire Wire Line
-	10200 6050 9350 6050
-Connection ~ 9300 3900
-Wire Wire Line
 	9350 4850 9750 4850
 Wire Wire Line
@@
 	9350 5550 9750 5550
 Wire Wire Line
-	6250 5700 7150 5700
-Wire Wire Line
-	7150 5700 7150 4100
-Wire Wire Line
 	7150 4100 7450 4100
-Wire Wire Line
-	9400 4100 9400 2700
-Wire Wire Line
-	9400 2700 9300 2700
-Wire Wire Line
-	7450 4100 9400 4100
-Wire Wire Line
-	9400 2700 10300 2700
-Wire Wire Line
-	10300 2700 10300 5950
-Wire Wire Line
-	10300 5950 9350 5950
-Connection ~ 9400 2700
 $Comp
 L power:VCC #PWR0109
@@
 	1    0    0    -1
 $EndComp
-NoConn ~ 6250 5300
 Wire Wire Line
 	5100 6000 5100 6400
 NoConn ~ 6250 5800
+Text Label 6250 5300 0    50   ~ 0
+LCE*
+Text Label 6250 5400 0    50   ~ 0
+LOE*
+Text Label 6250 5500 0    50   ~ 0
+UCE*
+Text Label 6250 5600 0    50   ~ 0
+UOE*
+NoConn ~ 6250 5700
 Wire Bus Line
 	6550 1700 7000 1700
@@
 Wire Bus Line
 	9850 1500 9850 5800
+Text GLabel 9300 2800 2    50   Input ~ 0
+WE0*
+Text GLabel 9350 6050 2    50   Input ~ 0
+WE1*
+Text Label 9350 5850 0    50   ~ 0
+UCE*
+Text Label 9350 5950 0    50   ~ 0
+UOE*
+Text Label 9300 2600 0    50   ~ 0
+LCE*
+Text Label 9300 2700 0    50   ~ 0
+LOE*
 $EndSCHEMATC
